Commit message: tool and psm integrated sdf

File: dvrk_model/PSM/PSM.urdf (robot description, URDF)
Before this commit: robot PSM, 13 links, 12 joints
Links:
- link base_link: geometry collision mesh filename=package://dvrk_model/PSM/meshes/base_link.STL; visual mesh filename=package://dvrk_model/PSM/meshes/base_link.STL
- link main_insertion_Link: geometry collision mesh filename=package://dvrk_model/PSM/meshes/main_insertion_Link.STL; visual mesh filename=package://dvrk_model/PSM/meshes/main_insertion_Link.STL
- link pitch_back_Link: geometry collision mesh filename=package://dvrk_model/PSM/meshes/pitch_back_Link.STL; visual mesh filename=package://dvrk_model/PSM/meshes/pitch_back_Link.STL
- link pitch_bottom_Link: geometry collision mesh filename=package://dvrk_model/PSM/meshes/pitch_bottom_Link.STL; visual mesh filename=package://dvrk_model/PSM/meshes/pitch_bottom_Link.STL
- link pitch_end_Link: geometry collision mesh filename=package://dvrk_model/PSM/meshes/pitch_end_Link.STL; visual mesh filename=package://dvrk_model/PSM/meshes/pitch_end_Link.STL
- link pitch_front_Link: geometry collision mesh filename=package://dvrk_model/PSM/meshes/pitch_front_Link.STL; visual mesh filename=package://dvrk_model/PSM/meshes/pitch_front_Link.STL
- link pitch_top_Link: geometry collision mesh filename=package://dvrk_model/PSM/meshes/pitch_top_Link.STL; visual mesh filename=package://dvrk_model/PSM/meshes/pitch_top_Link.STL
- link tool_gripper1_link: geometry collision mesh filename=package://dvrk_model/PSM/meshes/tool_gripper1_link.STL; visual mesh filename=package://dvrk_model/PSM/meshes/tool_gripper1_link.STL
- link tool_gripper2_link: geometry collision mesh filename=package://dvrk_model/PSM/meshes/tool_gripper2_link.STL; visual mesh filename=package://dvrk_model/PSM/meshes/tool_gripper2_link.STL
- link tool_pitch_link: geometry collision mesh filename=package://dvrk_model/PSM/meshes/tool_pitch_link.STL; visual mesh filename=package://dvrk_model/PSM/meshes/tool_pitch_link.STL
- link tool_roll_link: geometry collision mesh filename=package://dvrk_model/PSM/meshes/tool_roll_link.STL; visual mesh filename=package://dvrk_model/PSM/meshes/tool_roll_link.STL
- link tool_yaw_link: geometry collision mesh filename=package://dvrk_model/PSM/meshes/tool_yaw_link.STL; visual mesh filename=package://dvrk_model/PSM/meshes/tool_yaw_link.STL
- link yaw_Link: geometry collision mesh filename=package://dvrk_model/PSM/meshes/yaw_Link.STL; visual mesh filename=package://dvrk_model/PSM/meshes/yaw_Link.STL
Joints:
- joint main_insertion_joint: limit (none) -> lower=0 upper=0.24 effort=1000 velocity=1
- joint pitch_back_joint: limit (none) -> lower=-0.93556 upper=0.94249 effort=1000 velocity=10; type continuous -> revolute
- joint pitch_bottom_joint: limit (none) -> lower=-0.94249 upper=0.93556 effort=1000 velocity=10; type continuous -> revolute
- joint pitch_end_joint: limit (none) -> lower=-0.93556 upper=0.94249 effort=1000 velocity=10; type continuous -> revolute
- joint pitch_front_joint: limit (none) -> lower=-0.93556 upper=0.94249 effort=1000 velocity=10; type continuous -> revolute
- joint pitch_top_joint: limit (none) -> lower=-0.94249 upper=0.93556 effort=1000 velocity=10; type continuous -> revolute
- joint tool_gripper1_joint: limit (none) -> lower=0 upper=1 effort=0 velocity=0; type continuous -> revolute
- joint tool_gripper2_joint: limit (none) -> lower=0 upper=1 effort=0 velocity=0; type continuous -> revolute
- joint tool_pitch_joint: limit (none) -> lower=-1.5708 upper=1.5708 effort=1000 velocity=10; type continuous -> revolute
- joint tool_roll_joint: limit (none) -> lower=-3.14159 upper=3.14159 effort=1000 velocity=10; type continuous -> revolute
- joint tool_yaw_joint: limit (none) -> lower=-1.5708 upper=1.5708 effort=1000 velocity=10; type continuous -> revolute
- joint yaw_joint: limit (none) -> lower=-1.605 upper=1.5994 effort=1000 velocity=10; type continuous -> revolute
