Commit message: PSM Urdf

File: dvrk_model/PSM/psm.urdf.xacro (robot description, xacro)
@@ -17,8 +17,8 @@
     <inertial>
       <origin
-        xyz="-0.170155334863205 1.21879980786378E-08 0.066793166062727"
-        rpy="0 0 0" />
-      <mass
-        value="2.01611935350024" />
+        xyz="-1.2188E-08 -0.17016 -0.085607"
+        rpy="0 0 0" />
+      <mass
+        value="2.0161" />
       <inertia
         ixx="0"
@@ -40,5 +40,5 @@
         name="">
         <color
-          rgba="0.898039215686275 0.917647058823529 0.929411764705882 1" />
+          rgba="0.89804 0.91765 0.92941 1" />
       </material>
     </visual>
@@ -57,8 +57,8 @@
     <inertial>
       <origin
-        xyz="7.84810687552783E-05 -0.0387688268954186 -0.158996070278593"
-        rpy="0 0 0" />
-      <mass
-        value="1.47048370646334" />
+        xyz="-0.038769 7.8481E-05 0.041596"
+        rpy="0 0 0" />
+      <mass
+        value="1.4705" />
       <inertia
         ixx="0"
@@ -80,5 +80,5 @@
         name="">
         <color
-          rgba="0.898039215686275 0.917647058823529 0.929411764705882 1" />
+          rgba="0.89804 0.91765 0.92941 1" />
       </material>
     </visual>
@@ -97,6 +97,6 @@
     type="revolute">
     <origin
-      xyz="0.1174 0 0.1524"
-      rpy="1.57079632679489 0 1.5707963267949" />
+      xyz="0 0 0"
+      rpy="1.5708 -1.5708 0" />
     <parent
       link="${prefix}base_link" />
@@ -104,10 +104,10 @@
       link="${prefix}yaw_Link" />
     <axis
-      xyz="0 0 -1" />
+      xyz="0 0 1" />
     <limit
       lower="-1.605"
       upper="1.5994"
       effort="1000"
-      velocity="10" />
+	  velocity="10" />
   </joint>
   <link
@@ -115,8 +115,8 @@
     <inertial>
       <origin
-        xyz="-0.0121747017772931 -0.0368970293075621 3.52126111557088E-05"
-        rpy="0 0 0" />
-      <mass
-        value="0.995108878833389" />
+        xyz="-0.011651 -0.036241 3.5576E-05"
+        rpy="0 0 0" />
+      <mass
+        value="0.98494" />
       <inertia
         ixx="0"
@@ -138,5 +138,5 @@
         name="">
         <color
-          rgba="0.898039215686275 0.917647058823529 0.929411764705882 1" />
+          rgba="0.89804 0.91765 0.92941 1" />
       </material>
     </visual>
@@ -155,6 +155,6 @@
     type="revolute">
     <origin
-      xyz="0 0 -0.147"
-      rpy="1.5708 0.29073 1.5708" />
+      xyz="0 0 0.0296"
+      rpy="-1.5708 -0.29073 1.7787E-15" />
     <parent
       link="${prefix}yaw_Link" />
@@ -163,9 +163,9 @@
     <axis
       xyz="0 0 1" />
-    <limit
+	<limit
       lower="-0.93556"
       upper="0.94249"
       effort="1000"
-      velocity="10" />
+	  velocity="10" />
   </joint>
   <link
@@ -173,8 +173,8 @@
     <inertial>
       <origin
-        xyz="0.0103480348652787 0.256832099418565 -6.17918781630264E-06"
-        rpy="0 0 0" />
-      <mass
-        value="0.44569486685622" />
+        xyz="0.25683 -0.010348 -6.1792E-06"
+        rpy="0 0 0" />
+      <mass
+        value="0.44569" />
       <inertia
         ixx="0"
@@ -196,5 +196,5 @@
         name="">
         <color
-          rgba="0.898039215686275 0.917647058823529 0.929411764705882 1" />
+          rgba="0.89804 0.91765 0.92941 1" />
       </material>
     </visual>
@@ -214,5 +214,5 @@
     <origin
       xyz="0.15 0 0"
-      rpy="4.7846E-27 -1.6818E-39 0.29073" />
+      rpy="0 0 1.8615" />
     <parent
       link="${prefix}pitch_back_Link" />
@@ -225,5 +225,5 @@
       upper="0.93556"
       effort="1000"
-      velocity="10" />
+	  velocity="10" />
     <mimic joint="${prefix}pitch_back_joint" multiplier="-1"/>
   </joint>
@@ -232,8 +232,8 @@
     <inertial>
       <origin
-        xyz="0.136126867582571 -0.00192933659797534 -5.97041916218732E-08"
-        rpy="0 0 0" />
-      <mass
-        value="2.09102449600225" />
+        xyz="-0.0019293 -0.13613 -5.9688E-08"
+        rpy="0 0 0" />
+      <mass
+        value="2.091" />
       <inertia
         ixx="0"
@@ -255,5 +255,5 @@
         name="">
         <color
-          rgba="0.898039215686275 0.917647058823529 0.929411764705882 1" />
+          rgba="0.89804 0.91765 0.92941 1" />
       </material>
     </visual>
@@ -272,5 +272,5 @@
     type="revolute">
     <origin
-      xyz="0 0.516 0"
+      xyz="0.516 0 0"
       rpy="0 0 -3.5146E-13" />
     <parent
@@ -284,5 +284,5 @@
       upper="0.94249"
       effort="1000"
-      velocity="10" />
+	  velocity="10" />
     <mimic joint="${prefix}pitch_back_joint" multiplier="1"/>
   </joint>
@@ -291,20 +291,20 @@
     <inertial>
       <origin
-        xyz="0.0197642044936629 1.01697660725325E-13 -0.0117993612461738"
-        rpy="0 0 0" />
-      <mass
-        value="0.0311805666105664" />
-      <inertia
-        ixx="0"
-        ixy="0"
-        ixz="0"
-        iyy="0"
-        iyz="0"
-        izz="0" />
-    </inertial>
-    <visual>
-      <origin
-        xyz="0 0 0"
-        rpy="0 0 0" />
+        xyz="0.0040563 -0.00010934 0.0098616"
+        rpy="0 0 0" />
+      <mass
+        value="0.22491" />
+      <inertia
+        ixx="1.6985E-05"
+        ixy="-6.2173E-08"
+        ixz="1.2317E-05"
+        iyy="2.5916E-05"
+        iyz="8.5735E-08"
+        izz="8.9322E-06" />
+    </inertial>
+    <visual>
+      <origin
+        xyz="0 0 0"
+        rpy=" 0 0 1.5708" />
       <geometry>
         <mesh
@@ -314,5 +314,5 @@
         name="">
         <color
-          rgba="1 0.556862745098039 0.0588235294117647 0.4" />
+          rgba="1 0.55686 0.058824 0.4" />
       </material>
     </visual>
@@ -331,6 +331,6 @@
     type="prismatic">
     <origin
-      xyz="0.28809 0.043 0"
-      rpy="1.5708 1.1996E-14 -1.5708" />
+      xyz="0.043 -0.28809 0"
+      rpy="1.5708 1.5708 3.1416" />
     <parent
       link="${prefix}pitch_end_Link" />
@@ -343,5 +343,296 @@
       upper="0.24"
       effort="1000"
-      velocity="1" />
+	  velocity="1" />
+  </joint>
+  <link
+    name="${prefix}tool_roll_link">
+    <inertial>
+      <origin
+        xyz="-1.1313E-08 -7.4597E-09 -0.0058234"
+        rpy="0 0 0" />
+      <mass
+        value="0.00033225" />
+      <inertia
+        ixx="0"
+        ixy="0"
+        ixz="0"
+        iyy="0"
+        iyz="0"
+        izz="0" />
+    </inertial>
+    <visual>
+      <origin
+        xyz="0 0 1.5708"
+        rpy="0 0 0" />
+      <geometry>
+        <mesh
+          filename="package://dvrk_model/PSM/meshes/tool_roll_link.STL" />
+      </geometry>
+      <material
+        name="">
+        <color
+          rgba="0.79608 0.82353 0.93725 1" />
+      </material>
+    </visual>
+    <collision>
+      <origin
+        xyz="0 0 0"
+        rpy="0 0 0" />
+      <geometry>
+        <mesh
+          filename="package://dvrk_model/PSM/meshes/tool_roll_link.STL" />
+      </geometry>
+    </collision>
+  </link>
+  <joint
+    name="${prefix}tool_roll_joint"
+    type="revolute">
+    <origin
+      xyz="0 0 0.4162"
+      rpy="0 0 -1.5708" />
+    <parent
+      link="${prefix}main_insertion_Link" />
+    <child
+      link="${prefix}tool_roll_link" />
+    <axis
+      xyz="0 0 1" />
+    <limit
+      lower="-3.14159"
+      upper="3.14159"
+      effort="1000"
+      velocity="10" />
+  </joint>
+  <link
+    name="${prefix}tool_pitch_link">
+    <inertial>
+      <origin
+        xyz="0.0035763 -7.363E-08 4.4763E-06"
+        rpy="0 0 0" />
+      <mass
+        value="0.00025784" />
+      <inertia
+        ixx="1.2364E-13"
+        ixy="2.9238E-15"
+        ixz="4.1903E-12"
+        iyy="1.4213E-10"
+        iyz="-8.6271E-17"
+        izz="1.4201E-10" />
+    </inertial>
+    <visual>
+      <origin
+        xyz="0 0 0"
+        rpy="0 0 0" />
+      <geometry>
+        <mesh
+          filename="package://dvrk_model/PSM/meshes/tool_pitch_link.STL" />
+      </geometry>
+      <material
+        name="">
+        <color
+          rgba="0.79608 0.82353 0.93725 1" />
+      </material>
+    </visual>
+    <collision>
+      <origin
+        xyz="0 0 0"
+        rpy="0 0 0" />
+      <geometry>
+        <mesh
+          filename="package://dvrk_model/PSM/meshes/tool_pitch_link.STL" />
+      </geometry>
+    </collision>
+  </link>
+  <joint
+    name="${prefix}tool_pitch_joint"
+    type="revolute">
+    <origin
+      xyz="0 0 0"
+      rpy="1.5708 -1.5708 3.1416" />
+    <parent
+      link="${prefix}tool_roll_link" />
+    <child
+      link="${prefix}tool_pitch_link" />
+    <axis
+      xyz="0 0 1" />
+    <limit
+      lower="-1.5708"
+      upper="1.5708"
+      effort="1000"
+      velocity="10" />
+  </joint>
+  <link
+    name="${prefix}tool_yaw_link">
+    <inertial>
+      <origin
+        xyz="-1.0567E-14 -2.3287E-14 -5E-05"
+        rpy="0 0 0" />
+      <mass
+        value="6.6366E-06" />
+      <inertia
+        ixx="0"
+        ixy="0"
+        ixz="0"
+        iyy="0"
+        iyz="0"
+        izz="0" />
+    </inertial>
+    <visual>
+      <origin
+        xyz="0 0 0"
+        rpy="0 0 0" />
+      <geometry>
+        <mesh
+          filename="package://dvrk_model/PSM/meshes/tool_yaw_link.STL" />
+      </geometry>
+      <material
+        name="">
+        <color
+          rgba="0.79608 0.82353 0.93725 1" />
+      </material>
+    </visual>
+    <collision>
+      <origin
+        xyz="0 0 0"
+        rpy="0 0 0" />
+      <geometry>
+        <mesh
+          filename="package://dvrk_model/PSM/meshes/tool_yaw_link.STL" />
+      </geometry>
+    </collision>
+  </link>
+  <joint
+    name="${prefix}tool_yaw_joint"
+    type="revolute">
+    <origin
+      xyz="0.0091 0 0"
+      rpy="1.5708 -1.5708 3.1416" />
+    <parent
+      link="${prefix}tool_pitch_link" />
+    <child
+      link="${prefix}tool_yaw_link" />
+    <axis
+      xyz="0 0 1" />
+    <limit
+      lower="-1.5708"
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
Commit message: Removed unnecessarily long scientific precision that should be zeros

File: dvrk_model/PSM/psm.urdf.xacro (robot description, xacro)
@@ -17,5 +17,5 @@
     <inertial>
       <origin
-        xyz="-1.2188E-08 -0.17016 -0.085607"
+        xyz="0 -0.17016 -0.085607"
         rpy="0 0 0" />
       <mass
@@ -57,5 +57,5 @@
     <inertial>
       <origin
-        xyz="-0.038769 7.8481E-05 0.041596"
+        xyz="-0.038769 0 0.041596"
         rpy="0 0 0" />
       <mass
@@ -115,5 +115,5 @@
     <inertial>
       <origin
-        xyz="-0.011651 -0.036241 3.5576E-05"
+        xyz="-0.011651 -0.036241 0"
         rpy="0 0 0" />
       <mass
@@ -156,5 +156,5 @@
     <origin
       xyz="0 0 0.0296"
-      rpy="-1.5708 -0.29073 1.7787E-15" />
+      rpy="-1.5708 -0.29073 0" />
     <parent
       link="${prefix}yaw_Link" />
@@ -173,5 +173,5 @@
     <inertial>
       <origin
-        xyz="0.25683 -0.010348 -6.1792E-06"
+        xyz="0.25683 -0.010348 0"
         rpy="0 0 0" />
       <mass
@@ -232,5 +232,5 @@
     <inertial>
       <origin
-        xyz="-0.0019293 -0.13613 -5.9688E-08"
+        xyz="-0.0019293 -0.13613 0"
         rpy="0 0 0" />
       <mass
@@ -273,5 +273,5 @@
     <origin
       xyz="0.516 0 0"
-      rpy="0 0 -3.5146E-13" />
+      rpy="0 0 0" />
     <parent
       link="${prefix}pitch_bottom_Link" />
@@ -296,15 +296,15 @@
         value="0.22491" />
       <inertia
-        ixx="1.6985E-05"
-        ixy="-6.2173E-08"
-        ixz="1.2317E-05"
-        iyy="2.5916E-05"
-        iyz="8.5735E-08"
-        izz="8.9322E-06" />
-    </inertial>
-    <visual>
-      <origin
-        xyz="0 0 0"
-        rpy=" 0 0 1.5708" />
+        ixx="0"
+        ixy="0"
+        ixz="0"
+        iyy="0"
+        iyz="0"
+        izz="0" />
+    </inertial>
+    <visual>
+      <origin
+        xyz="0 0 0"
+        rpy="0 0 1.5708" />
       <geometry>
         <mesh
@@ -349,5 +349,5 @@
     <inertial>
       <origin
-        xyz="-1.1313E-08 -7.4597E-09 -0.0058234"
+        xyz="0 0 -0.0058234"
         rpy="0 0 0" />
       <mass
@@ -407,15 +407,15 @@
     <inertial>
       <origin
-        xyz="0.0035763 -7.363E-08 4.4763E-06"
+        xyz="0.0035763 0 0"
         rpy="0 0 0" />
       <mass
         value="0.00025784" />
       <inertia
-        ixx="1.2364E-13"
-        ixy="2.9238E-15"
-        ixz="4.1903E-12"
-        iyy="1.4213E-10"
-        iyz="-8.6271E-17"
-        izz="1.4201E-10" />
+        ixx="0"
+        ixy="0"
+        ixz="0"
+        iyy="0"
+        iyz="0"
+        izz="0" />
     </inertial>
     <visual>
@@ -465,8 +465,8 @@
     <inertial>
       <origin
-        xyz="-1.0567E-14 -2.3287E-14 -5E-05"
-        rpy="0 0 0" />
-      <mass
-        value="6.6366E-06" />
+        xyz="0 0 0"
+        rpy="0 0 0" />
+      <mass
+        value="0" />
       <inertia
         ixx="0"
@@ -526,5 +526,5 @@
         rpy="0 0 0" />
       <mass
-        value="3.7467E-05" />
+        value="0" />
       <inertia
         ixx="0"
@@ -585,5 +585,5 @@
         rpy="0 0 0" />
       <mass
-        value="3.7467E-05" />
+        value="0" />
       <inertia
         ixx="0"
@@ -640,5 +640,5 @@
     <inertial>
       <origin
-        xyz="0.31246 -0.00056566 -3.4131E-07"
+        xyz="0.31246 -0.00056566 0"
         rpy="0 0 0" />
       <mass
@@ -699,5 +699,5 @@
     <inertial>
       <origin
-        xyz="0.096269 1.1116E-12 0.047551"
+        xyz="0.096269 0 0.047551"
         rpy="0 0 0" />
       <mass
@@ -740,5 +740,5 @@
     <origin
       xyz="0 0 -0.0664"
-      rpy="-1.5708 -0.29073 1.7787E-15" />
+      rpy="-1.5708 -0.29073 0" />
     <parent
       link="${prefix}yaw_Link" />
