Commit message: new model, new package

File: PSM/urdf/PSM.urdf (robot description, URDF)
Before this commit: robot PSM, 13 links, 12 joints
Links:
- link pitch_back_Link: mass 0.99511 -> 0.98494
- link tool_gripper1_link: mass 3.907E-05 -> 3.7467E-05
- link tool_gripper2_link: mass 3.907E-05 -> 3.7467E-05
- link tool_pitch_link: mass 0.00025977 -> 0.00025784
Joints:
- joint main_insertion_joint: limit (none) -> effort=0 velocity=0; origin xyz=0.0430000000019171 -0.288089999999913 0 rpy=1.5707963267949 0 3.14159265358979 -> xyz=0.043 -0.28809 0 rpy=1.5708 0 3.1416
- joint pitch_back_joint: origin xyz=0 0 0.0295999999999997 rpy=-1.5707963267949 -0.290727597908961 1.77865254633244E-15 -> xyz=0 0 0.0296 rpy=-1.5708 -0.29073 1.7787E-15
- joint pitch_front_joint: origin xyz=0 0 -0.0664000000000003 rpy=-1.57079632679489 -0.290727597908941 1.77865254633244E-15 -> xyz=0 0 -0.0664 rpy=-1.5708 -0.29073 1.7787E-15
- joint pitch_top_joint: origin xyz=0.183657966666658 0.0141205977162999 0 rpy=0 0 1.86152392470386 -> xyz=0.18366 0.014121 0 rpy=0 0 1.8615
- joint tool_gripper1_joint: origin xyz=0 0 0 rpy=0 0 1.7432292974031E-33 -> xyz=0 0 0 rpy=0 0 0
- joint tool_gripper2_joint: origin xyz=0 0 0 rpy=0 0 1.7432292974031E-33 -> xyz=0 0 0 rpy=0 0 0
- joint tool_pitch_joint: origin xyz=0 0 0 rpy=1.5707963267949 -1.5707963267949 0 -> xyz=0 0 0 rpy=1.5708 -1.5708 0
- joint tool_roll_joint: origin xyz=0 0 0.416199999999902 rpy=0 0 3.14159265358979 -> xyz=0 0 0.4162 rpy=0 0 3.1416
- joint tool_yaw_joint: origin xyz=0.00910000000003011 -5.00000000686063E-05 0 rpy=1.57079632679486 -1.5707963267949 0 -> xyz=0.0091 0 0 rpy=1.5708 -1.5708 0
- joint yaw_joint: origin xyz=0 0 0 rpy=1.57079632679489 -1.5707963267949 0 -> xyz=0 0 0 rpy=1.5708 -1.5708 0
