Commit message: rename cart to suj, added .yaml's, cleaned launch files

File: dvrk_description/ecm/ecm.urdf.xacro (robot description, xacro)
@@ -7,9 +7,9 @@
     <joint name="fixed_joint" type="fixed">
       <parent link="${parent_link}"/>
-      <child link="${prefix}_base_link"/>
+      <child link="${prefix}base_link"/>
       <origin rpy="${rpy}" xyz="${xyz}"/>
     </joint>
     <link
-      name="${prefix}_base_link">
+      name="${prefix}base_link">
       <inertial>
         <origin
@@ -51,5 +51,5 @@
     </link>
     <link
-      name="${prefix}_yaw_link">
+      name="${prefix}yaw_link">
       <inertial>
         <origin
@@ -91,5 +91,5 @@
     </link>
     <joint
-      name="${prefix}_yaw_joint"
+      name="${prefix}yaw_joint"
       type="revolute">
       <origin
@@ -97,7 +97,7 @@
         rpy="1.57079632679615 -3.58046925441613E-13 1.5707963267949" />
       <parent
-        link="${prefix}_base_link" />
-      <child
-        link="${prefix}_yaw_link" />
+        link="${prefix}base_link" />
+      <child
+        link="${prefix}yaw_link" />
       <axis
         xyz="0 0 1" />
@@ -109,5 +109,5 @@
     </joint>
     <link
-      name="${prefix}_pitch_front_link">
+      name="${prefix}pitch_front_link">
       <inertial>
         <origin
@@ -149,5 +149,5 @@
     </link>
     <joint
-      name="${prefix}_pitch_front_joint"
+      name="${prefix}pitch_front_joint"
       type="revolute">
       <origin
@@ -155,7 +155,7 @@
         rpy="3.14 -1.5707963267949 0" />
       <parent
-        link="${prefix}_yaw_link" />
-      <child
-        link="${prefix}_pitch_front_link" />
+        link="${prefix}yaw_link" />
+      <child
+        link="${prefix}pitch_front_link" />
       <axis
         xyz="0 0 1" />
@@ -167,5 +167,5 @@
     </joint>
     <link
-      name="${prefix}_pitch_bottom_link">
+      name="${prefix}pitch_bottom_link">
       <inertial>
         <origin
@@ -207,5 +207,5 @@
     </link>
     <joint
-      name="${prefix}_pitch_bottom_joint"
+      name="${prefix}pitch_bottom_joint"
       type="revolute">
       <origin
@@ -213,7 +213,7 @@
         rpy="0 0 0" />
       <parent
-        link="${prefix}_pitch_front_link" />
-      <child
-        link="${prefix}_pitch_bottom_link" />
+        link="${prefix}pitch_front_link" />
+      <child
+        link="${prefix}pitch_bottom_link" />
       <axis
         xyz="0 0 1" />
@@ -223,8 +223,8 @@
         effort="1000"
         velocity="10" />
-      <mimic joint="${prefix}_pitch_front_joint" multiplier="-1"/>
-    </joint>
-    <link
-      name="${prefix}_pitch_end_link">
+      <mimic joint="${prefix}pitch_front_joint" multiplier="-1"/>
+    </joint>
+    <link
+      name="${prefix}pitch_end_link">
       <inertial>
         <origin
@@ -266,5 +266,5 @@
     </link>
     <joint
-      name="${prefix}_pitch_end_joint"
+      name="${prefix}pitch_end_joint"
       type="revolute">
       <origin
@@ -272,7 +272,7 @@
         rpy="0 0 0" />
       <parent
-        link="${prefix}_pitch_bottom_link" />
-      <child
-        link="${prefix}_pitch_end_link" />
+        link="${prefix}pitch_bottom_link" />
+      <child
+        link="${prefix}pitch_end_link" />
       <axis
         xyz="0 0 1" />
@@ -282,8 +282,8 @@
         effort="1000"
         velocity="10" />
-      <mimic joint="${prefix}_pitch_front_joint" multiplier="1"/>
-    </joint>
-    <link
-      name="${prefix}_main_insertion_link">
+      <mimic joint="${prefix}pitch_front_joint" multiplier="1"/>
+    </joint>
+    <link
+      name="${prefix}main_insertion_link">
       <inertial>
         <origin
@@ -325,5 +325,5 @@
     </link>
     <joint
-      name="${prefix}_main_insertion_joint"
+      name="${prefix}main_insertion_joint"
       type="prismatic">
       <origin
@@ -331,7 +331,7 @@
         rpy="-1.5708 0 0" />
       <parent
-        link="${prefix}_pitch_end_link" />
-      <child
-        link="${prefix}_main_insertion_link" />
+        link="${prefix}pitch_end_link" />
+      <child
+        link="${prefix}main_insertion_link" />
       <axis
         xyz="0 0 1" />
@@ -343,5 +343,5 @@
     </joint>
     <link
-      name="${prefix}_tool_link">
+      name="${prefix}tool_link">
       <inertial>
         <origin
@@ -383,5 +383,5 @@
     </link>
     <joint
-      name="${prefix}_tool_joint"
+      name="${prefix}tool_joint"
       type="revolute">
       <origin
@@ -389,7 +389,7 @@
         rpy="0 0 0" />
       <parent
-        link="${prefix}_main_insertion_link" />
-      <child
-        link="${prefix}_tool_link" />
+        link="${prefix}main_insertion_link" />
+      <child
+        link="${prefix}tool_link" />
       <axis
         xyz="0 0 -1" />
@@ -401,5 +401,5 @@
     </joint>
     <link
-      name="${prefix}_pitch_top_link">
+      name="${prefix}pitch_top_link">
       <inertial>
         <origin
@@ -441,5 +441,5 @@
     </link>
     <joint
-      name="${prefix}_pitch_top_joint"
+      name="${prefix}pitch_top_joint"
       type="revolute">
       <origin
@@ -447,7 +447,7 @@
         rpy="0 0 0" />
       <parent
-        link="${prefix}_pitch_front_link" />
-      <child
-        link="${prefix}_pitch_top_link" />
+        link="${prefix}pitch_front_link" />
+      <child
+        link="${prefix}pitch_top_link" />
       <axis
         xyz="0 0 1" />
@@ -457,8 +457,8 @@
         effort="1000"
         velocity="10" />
-      <mimic joint="${prefix}_pitch_front_joint" multiplier="-1"/>
-    </joint>
-    <link
-      name="${prefix}_pitch_back_link">
+      <mimic joint="${prefix}pitch_front_joint" multiplier="-1"/>
+    </joint>
+    <link
+      name="${prefix}pitch_back_link">
       <inertial>
         <origin
@@ -500,5 +500,5 @@
     </link>
     <joint
-      name="${prefix}_pitch_back_joint"
+      name="${prefix}pitch_back_joint"
       type="revolute">
       <origin
@@ -506,7 +506,7 @@
         rpy="3.14 -1.5707963267949 0" />
       <parent
-        link="${prefix}_yaw_link" />
-      <child
-        link="${prefix}_pitch_back_link" />
+        link="${prefix}yaw_link" />
+      <child
+        link="${prefix}pitch_back_link" />
       <axis
         xyz="0 0 1" />
@@ -516,8 +516,8 @@
         effort="1000"
         velocity="10" />
-      <mimic joint="${prefix}_pitch_front_joint" multiplier="1"/>
-    </joint>
-    <link
-      name="${prefix}_remote_center_link">
+      <mimic joint="${prefix}pitch_front_joint" multiplier="1"/>
+    </joint>
+    <link
+      name="${prefix}remote_center_link">
       <inertial>
         <origin
@@ -559,5 +559,5 @@
     </link>
     <joint
-      name="${prefix}_remote_center_joint"
+      name="${prefix}remote_center_joint"
       type="fixed">
       <origin
@@ -565,13 +565,13 @@
         rpy="-1.249734375614E-12 3.58046925441613E-13 -1.5707963267949" />
       <parent
-        link="${prefix}_base_link" />
-      <child
-        link="${prefix}_remote_center_link" />
+        link="${prefix}base_link" />
+      <child
+        link="${prefix}remote_center_link" />
       <axis
         xyz="0 0 0" />
     </joint>
-    <link name="${prefix}_end_link"/>
-    <joint
-      name="${prefix}_end_joint"
+    <link name="${prefix}end_link"/>
+    <joint
+      name="${prefix}end_joint"
       type="fixed">
       <origin
@@ -579,7 +579,7 @@
         rpy="0 0 0" />
       <parent
-        link="${prefix}_tool_link" />
-      <child
-        link="${prefix}_end_link" />
+        link="${prefix}tool_link" />
+      <child
+        link="${prefix}end_link" />
       <axis
         xyz="0 0 0" />

File: dvrk_description/suj/suj.xacro (robot description, xacro)
@@ -34,5 +34,5 @@
       <geometry>
         <mesh
-          filename="package://dvrk_description/cart/meshes/base_link.STL" />
+          filename="package://dvrk_description/suj/meshes/base_link.STL" />
       </geometry>
       <material
@@ -48,5 +48,5 @@
       <geometry>
         <mesh
-          filename="package://dvrk_description/cart/meshes/base_link.STL" />
+          filename="package://dvrk_description/suj/meshes/base_link.STL" />
       </geometry>
     </collision>
@@ -74,19 +74,19 @@
       <geometry>
         <mesh
-          filename="package://dvrk_description/cart/meshes/suj_psm2_L0.STL" />
-      </geometry>
-      <material
-        name="">
-        <color
-          rgba="0.792156862745098 0.819607843137255 0.933333333333333 1" />
-      </material>
-    </visual>
-    <collision>
-      <origin
-        xyz="0 0 0"
-        rpy="0 0 0" />
-      <geometry>
-        <mesh
-          filename="package://dvrk_description/cart/meshes/suj_psm2_L0.STL" />
+          filename="package://dvrk_description/suj/meshes/suj_psm2_L0.STL" />
+      </geometry>
+      <material
+        name="">
+        <color
+          rgba="0.792156862745098 0.819607843137255 0.933333333333333 1" />
+      </material>
+    </visual>
+    <collision>
+      <origin
+        xyz="0 0 0"
+        rpy="0 0 0" />
+      <geometry>
+        <mesh
+          filename="package://dvrk_description/suj/meshes/suj_psm2_L0.STL" />
       </geometry>
     </collision>
@@ -132,19 +132,19 @@
       <geometry>
         <mesh
-          filename="package://dvrk_description/cart/meshes/suj_psm2_L1.STL" />
-      </geometry>
-      <material
-        name="">
-        <color
-          rgba="0.792156862745098 0.819607843137255 0.933333333333333 1" />
-      </material>
-    </visual>
-    <collision>
-      <origin
-        xyz="0 0 0"
-        rpy="0 0 0" />
-      <geometry>
-        <mesh
-          filename="package://dvrk_description/cart/meshes/suj_psm2_L1.STL" />
+          filename="package://dvrk_description/suj/meshes/suj_psm2_L1.STL" />
+      </geometry>
+      <material
+        name="">
+        <color
+          rgba="0.792156862745098 0.819607843137255 0.933333333333333 1" />
+      </material>
+    </visual>
+    <collision>
+      <origin
+        xyz="0 0 0"
+        rpy="0 0 0" />
+      <geometry>
+        <mesh
+          filename="package://dvrk_description/suj/meshes/suj_psm2_L1.STL" />
       </geometry>
     </collision>
@@ -185,19 +185,19 @@
       <geometry>
         <mesh
-          filename="package://dvrk_description/cart/meshes/suj_psm2_L2.STL" />
-      </geometry>
-      <material
-        name="">
-        <color
-          rgba="0.792156862745098 0.819607843137255 0.933333333333333 1" />
-      </material>
-    </visual>
-    <collision>
-      <origin
-        xyz="0 0 0"
-        rpy="0 0 0" />
-      <geometry>
-        <mesh
-          filename="package://dvrk_description/cart/meshes/suj_psm2_L2.STL" />
+          filename="package://dvrk_description/suj/meshes/suj_psm2_L2.STL" />
+      </geometry>
+      <material
+        name="">
+        <color
+          rgba="0.792156862745098 0.819607843137255 0.933333333333333 1" />
+      </material>
+    </visual>
+    <collision>
+      <origin
+        xyz="0 0 0"
+        rpy="0 0 0" />
+      <geometry>
+        <mesh
+          filename="package://dvrk_description/suj/meshes/suj_psm2_L2.STL" />
       </geometry>
     </collision>
@@ -238,19 +238,19 @@
       <geometry>
         <mesh
-          filename="package://dvrk_description/cart/meshes/suj_psm2_L3.STL" />
-      </geometry>
-      <material
-        name="">
-        <color
-          rgba="0.792156862745098 0.819607843137255 0.933333333333333 1" />
-      </material>
-    </visual>
-    <collision>
-      <origin
-        xyz="0 0 0"
-        rpy="0 0 0" />
-      <geometry>
-        <mesh
-          filename="package://dvrk_description/cart/meshes/suj_psm2_L3.STL" />
+          filename="package://dvrk_description/suj/meshes/suj_psm2_L3.STL" />
+      </geometry>
+      <material
+        name="">
+        <color
+          rgba="0.792156862745098 0.819607843137255 0.933333333333333 1" />
+      </material>
+    </visual>
+    <collision>
+      <origin
+        xyz="0 0 0"
+        rpy="0 0 0" />
+      <geometry>
+        <mesh
+          filename="package://dvrk_description/suj/meshes/suj_psm2_L3.STL" />
       </geometry>
     </collision>
@@ -291,19 +291,19 @@
       <geometry>
         <mesh
-          filename="package://dvrk_description/cart/meshes/suj_psm2_L4.STL" />
-      </geometry>
-      <material
-        name="">
-        <color
-          rgba="0.792156862745098 0.819607843137255 0.933333333333333 1" />
-      </material>
-    </visual>
-    <collision>
-      <origin
-        xyz="0 0 0"
-        rpy="0 0 0" />
-      <geometry>
-        <mesh
-          filename="package://dvrk_description/cart/meshes/suj_psm2_L4.STL" />
+          filename="package://dvrk_description/suj/meshes/suj_psm2_L4.STL" />
+      </geometry>
+      <material
+        name="">
+        <color
+          rgba="0.792156862745098 0.819607843137255 0.933333333333333 1" />
+      </material>
+    </visual>
+    <collision>
+      <origin
+        xyz="0 0 0"
+        rpy="0 0 0" />
+      <geometry>
+        <mesh
+          filename="package://dvrk_description/suj/meshes/suj_psm2_L4.STL" />
       </geometry>
     </collision>
@@ -344,19 +344,19 @@
       <geometry>
         <mesh
-          filename="package://dvrk_description/cart/meshes/suj_ecm_L0.STL" />
-      </geometry>
-      <material
-        name="">
-        <color
-          rgba="0.792156862745098 0.819607843137255 0.933333333333333 1" />
-      </material>
-    </visual>
-    <collision>
-      <origin
-        xyz="0 0 0"
-        rpy="0 0 0" />
-      <geometry>
-        <mesh
-          filename="package://dvrk_description/cart/meshes/suj_ecm_L0.STL" />
+          filename="package://dvrk_description/suj/meshes/suj_ecm_L0.STL" />
+      </geometry>
+      <material
+        name="">
+        <color
+          rgba="0.792156862745098 0.819607843137255 0.933333333333333 1" />
+      </material>
+    </visual>
+    <collision>
+      <origin
+        xyz="0 0 0"
+        rpy="0 0 0" />
+      <geometry>
+        <mesh
+          filename="package://dvrk_description/suj/meshes/suj_ecm_L0.STL" />
       </geometry>
     </collision>
@@ -402,19 +402,19 @@
       <geometry>
         <mesh
-          filename="package://dvrk_description/cart/meshes/suj_ecm_L1.STL" />
-      </geometry>
-      <material
-        name="">
-        <color
-          rgba="0.792156862745098 0.819607843137255 0.933333333333333 1" />
-      </material>
-    </visual>
-    <collision>
-      <origin
-        xyz="0 0 0"
-        rpy="0 0 0" />
-      <geometry>
-        <mesh
-          filename="package://dvrk_description/cart/meshes/suj_ecm_L1.STL" />
+          filename="package://dvrk_description/suj/meshes/suj_ecm_L1.STL" />
+      </geometry>
+      <material
+        name="">
+        <color
+          rgba="0.792156862745098 0.819607843137255 0.933333333333333 1" />
+      </material>
+    </visual>
+    <collision>
+      <origin
+        xyz="0 0 0"
+        rpy="0 0 0" />
+      <geometry>
+        <mesh
+          filename="package://dvrk_description/suj/meshes/suj_ecm_L1.STL" />
       </geometry>
     </collision>
@@ -455,19 +455,19 @@
       <geometry>
         <mesh
-          filename="package://dvrk_description/cart/meshes/suj_ecm_L2.STL" />
-      </geometry>
-      <material
-        name="">
-        <color
-          rgba="0.792156862745098 0.819607843137255 0.933333333333333 1" />
-      </material>
-    </visual>
-    <collision>
-      <origin
-        xyz="0 0 0"
-        rpy="0 0 0" />
-      <geometry>
-        <mesh
-          filename="package://dvrk_description/cart/meshes/suj_ecm_L2.STL" />
+          filename="package://dvrk_description/suj/meshes/suj_ecm_L2.STL" />
+      </geometry>
+      <material
+        name="">
+        <color
+          rgba="0.792156862745098 0.819607843137255 0.933333333333333 1" />
+      </material>
+    </visual>
+    <collision>
+      <origin
+        xyz="0 0 0"
+        rpy="0 0 0" />
+      <geometry>
+        <mesh
+          filename="package://dvrk_description/suj/meshes/suj_ecm_L2.STL" />
       </geometry>
     </collision>
@@ -508,19 +508,19 @@
       <geometry>
         <mesh
-          filename="package://dvrk_description/cart/meshes/suj_ecm_L3.STL" />
-      </geometry>
-      <material
-        name="">
-        <color
-          rgba="0.792156862745098 0.819607843137255 0.933333333333333 1" />
-      </material>
-    </visual>
-    <collision>
-      <origin
-        xyz="0 0 0"
-        rpy="0 0 0" />
-      <geometry>
-        <mesh
-          filename="package://dvrk_description/cart/meshes/suj_ecm_L3.STL" />
+          filename="package://dvrk_description/suj/meshes/suj_ecm_L3.STL" />
+      </geometry>
+      <material
+        name="">
+        <color
+          rgba="0.792156862745098 0.819607843137255 0.933333333333333 1" />
+      </material>
+    </visual>
+    <collision>
+      <origin
+        xyz="0 0 0"
+        rpy="0 0 0" />
+      <geometry>
+        <mesh
+          filename="package://dvrk_description/suj/meshes/suj_ecm_L3.STL" />
       </geometry>
     </collision>
@@ -561,19 +561,19 @@
       <geometry>
         <mesh
-          filename="package://dvrk_description/cart/meshes/suj_psm1_L0.STL" />
-      </geometry>
-      <material
-        name="">
-        <color
-          rgba="0.792156862745098 0.819607843137255 0.933333333333333 1" />
-      </material>
-    </visual>
-    <collision>
-      <origin
-        xyz="0 0 0"
-        rpy="0 0 0" />
-      <geometry>
-        <mesh
-          filename="package://dvrk_description/cart/meshes/suj_psm1_L0.STL" />
+          filename="package://dvrk_description/suj/meshes/suj_psm1_L0.STL" />
+      </geometry>
+      <material
+        name="">
+        <color
+          rgba="0.792156862745098 0.819607843137255 0.933333333333333 1" />
+      </material>
+    </visual>
+    <collision>
+      <origin
+        xyz="0 0 0"
+        rpy="0 0 0" />
+      <geometry>
+        <mesh
+          filename="package://dvrk_description/suj/meshes/suj_psm1_L0.STL" />
       </geometry>
     </collision>
@@ -619,19 +619,19 @@
       <geometry>
         <mesh
-          filename="package://dvrk_description/cart/meshes/suj_psm1_L1.STL" />
-      </geometry>
-      <material
-        name="">
-        <color
-          rgba="0.792156862745098 0.819607843137255 0.933333333333333 1" />
-      </material>
-    </visual>
-    <collision>
-      <origin
-        xyz="0 0 0"
-        rpy="0 0 0" />
-      <geometry>
-        <mesh
-          filename="package://dvrk_description/cart/meshes/suj_psm1_L1.STL" />
+          filename="package://dvrk_description/suj/meshes/suj_psm1_L1.STL" />
+      </geometry>
+      <material
+        name="">
+        <color
+          rgba="0.792156862745098 0.819607843137255 0.933333333333333 1" />
+      </material>
+    </visual>
+    <collision>
+      <origin
+        xyz="0 0 0"
+        rpy="0 0 0" />
+      <geometry>
+        <mesh
+          filename="package://dvrk_description/suj/meshes/suj_psm1_L1.STL" />
       </geometry>
     </collision>
@@ -672,19 +672,19 @@
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