Commit message: The changes are summed below
1. Consistency in file naming convention
2. Renamed .urdf files that were actually .xacro
3. Removed lingering .urdf files, they can be generated automatically
4. Simplified scientific precision that basically intends to be zero
5. Fixed cart to suj in CMakeList file

File: dvrk_description/dvrk/dvrk_launch.urdf.xacro (robot description, xacro)
@@ -2,5 +2,5 @@
 <robot name="master" xmlns:xacro="http://www.ros.org/wiki/xacro">
 <!-- Macros -->
-<xacro:include filename="$(find dvrk_description)/suj/suj.xacro"/>
+<xacro:include filename="$(find dvrk_description)/suj/suj.urdf.xacro"/>
 <xacro:include filename="$(find dvrk_description)/psm/psm.urdf.xacro"/>
 <xacro:include filename="$(find dvrk_description)/ecm/ecm.urdf.xacro"/>

File: dvrk_description/ecm/ecm.urdf.xacro (robot description, xacro)
@@ -14,5 +14,5 @@
       <inertial>
         <origin
-          xyz="-0.0048227 -2.9669E-05 0.068959"
+          xyz="-0.0048227 0 0.068959"
           rpy="0 0 0" />
         <mass
@@ -54,5 +54,5 @@
       <inertial>
         <origin
-          xyz="2.7532E-07 -0.029045 0.10669"
+          xyz="0 -0.029045 0.10669"
           rpy="0 0 0" />
         <mass
@@ -60,6 +60,6 @@
         <inertia
           ixx="0.00086598"
-          ixy="7.8532E-10"
-          ixz="2.5709E-09"
+          ixy="0"
+          ixz="0"
           iyy="0.0016561"
           iyz="-0.00015825"
@@ -95,5 +95,5 @@
       <origin
         xyz="0.0731999999999783 0 0.101460000000185"
-        rpy="1.57079632679615 -3.58046925441613E-13 1.5707963267949" />
+        rpy="1.57079632679615 0 1.5707963267949" />
       <parent
         link="${prefix}base_link" />
@@ -112,5 +112,5 @@
       <inertial>
         <origin
-          xyz="-0.030619 -0.13578 -5.7828E-08"
+          xyz="-0.030619 -0.13578 0"
           rpy="0 0 0" />
         <mass
@@ -177,7 +177,7 @@
           ixx="0.00023901"
           ixy="0.00022767"
-          ixz="-3.8706E-06"
+          ixz="0"
           iyy="0.0030096"
-          iyz="-7.279E-07"
+          iyz="0"
           izz="0.0029617" />
       </inertial>
@@ -346,5 +346,5 @@
       <inertial>
         <origin
-          xyz="2.6548E-14 -0.0007925 -0.10732"
+          xyz="0 -0.0007925 -0.10732"
           rpy="0 0 0" />
         <mass
@@ -404,5 +404,5 @@
       <inertial>
         <origin
-          xyz="0.1702 -6.7816E-05 0.0007925"
+          xyz="0.1702 0 0.0007925"
           rpy="0 0 0" />
         <mass
@@ -522,5 +522,5 @@
       <inertial>
         <origin
-          xyz="-1.1102E-16 0 0"
+          xyz="0 0 0"
           rpy="0 0 0" />
         <mass
@@ -563,5 +563,5 @@
       <origin
         xyz="0.612599207482277 0 0.10159534323531"
-        rpy="-1.249734375614E-12 3.58046925441613E-13 -1.5707963267949" />
+        rpy="0 0 -1.5707963267949" />
       <parent
         link="${prefix}base_link" />

File: dvrk_description/mtm/mtm_launch.urdf.xacro (robot description, xacro)
@@ -5,6 +5,6 @@
   <link name="world"/>
   <xacro:mtm
-      prefix="left_"
+      prefix="mtm_"
       parent_link="world"
-      xyz="-0.25 0.0 1.0" rpy="0.0 0.0 0.0"/>
+      xyz="0.0 0.0 1.0" rpy="0.0 0.0 0.0"/>
 </robot>

File: dvrk_description/psm/psm.urdf.xacro (robot description, xacro)
@@ -17,5 +17,5 @@
     <inertial>
       <origin
-        xyz="-1.2188E-08 -0.17016 -0.085607"
+        xyz="0 -0.17016 -0.085607"
         rpy="0 0 0" />
       <mass
@@ -57,5 +57,5 @@
     <inertial>
       <origin
-        xyz="-0.038769 7.8481E-05 0.041596"
+        xyz="-0.038769 0 0.041596"
         rpy="0 0 0" />
       <mass
@@ -115,5 +115,5 @@
     <inertial>
       <origin
-        xyz="-0.011651 -0.036241 3.5576E-05"
+        xyz="-0.011651 -0.036241 0"
         rpy="0 0 0" />
       <mass
@@ -156,5 +156,5 @@
     <origin
       xyz="0 0 0.0296"
-      rpy="-1.5708 -0.29073 1.7787E-15" />
+      rpy="-1.5708 -0.29073 0" />
     <parent
       link="${prefix}yaw_Link" />
@@ -173,5 +173,5 @@
     <inertial>
       <origin
-        xyz="0.25683 -0.010348 -6.1792E-06"
+        xyz="0.25683 -0.010348 0"
         rpy="0 0 0" />
       <mass
@@ -232,5 +232,5 @@
     <inertial>
       <origin
-        xyz="-0.0019293 -0.13613 -5.9688E-08"
+        xyz="-0.0019293 -0.13613 0"
         rpy="0 0 0" />
       <mass
@@ -273,5 +273,5 @@
     <origin
       xyz="0.516 0 0"
-      rpy="0 0 -3.5146E-13" />
+      rpy="0 0 0" />
     <parent
       link="${prefix}pitch_bottom_Link" />
@@ -296,15 +296,15 @@
         value="0.22491" />
       <inertia
-        ixx="1.6985E-05"
-        ixy="-6.2173E-08"
-        ixz="1.2317E-05"
-        iyy="2.5916E-05"
-        iyz="8.5735E-08"
-        izz="8.9322E-06" />
-    </inertial>
-    <visual>
-      <origin
-        xyz="0 0 0"
-        rpy=" 0 0 1.5708" />
+        ixx="0"
+        ixy="0"
+        ixz="0"
+        iyy="0"
+        iyz="0"
+        izz="0" />
+    </inertial>
+    <visual>
+      <origin
+        xyz="0 0 0"
+        rpy="0 0 1.5708" />
       <geometry>
         <mesh
@@ -349,5 +349,5 @@
     <inertial>
       <origin
-        xyz="-1.1313E-08 -7.4597E-09 -0.0058234"
+        xyz="0 0 -0.0058234"
         rpy="0 0 0" />
       <mass
@@ -407,15 +407,15 @@
     <inertial>
       <origin
-        xyz="0.0035763 -7.363E-08 4.4763E-06"
+        xyz="0.0035763 0 0"
         rpy="0 0 0" />
       <mass
         value="0.00025784" />
       <inertia
-        ixx="1.2364E-13"
-        ixy="2.9238E-15"
-        ixz="4.1903E-12"
-        iyy="1.4213E-10"
-        iyz="-8.6271E-17"
-        izz="1.4201E-10" />
+        ixx="0"
+        ixy="0"
+        ixz="0"
+        iyy="0"
+        iyz="0"
+        izz="0" />
     </inertial>
     <visual>
@@ -465,8 +465,8 @@
     <inertial>
       <origin
-        xyz="-1.0567E-14 -2.3287E-14 -5E-05"
-        rpy="0 0 0" />
-      <mass
-        value="6.6366E-06" />
+        xyz="0 0 0"
+        rpy="0 0 0" />
+      <mass
+        value="0" />
       <inertia
         ixx="0"
@@ -526,5 +526,5 @@
         rpy="0 0 0" />
       <mass
-        value="3.7467E-05" />
+        value="0" />
       <inertia
         ixx="0"
@@ -585,5 +585,5 @@
         rpy="0 0 0" />
       <mass
-        value="3.7467E-05" />
+        value="0" />
       <inertia
         ixx="0"
@@ -640,5 +640,5 @@
     <inertial>
       <origin
-        xyz="0.31246 -0.00056566 -3.4131E-07"
+        xyz="0.31246 -0.00056566 0"
         rpy="0 0 0" />
       <mass
@@ -699,5 +699,5 @@
     <inertial>
       <origin
-        xyz="0.096269 1.1116E-12 0.047551"
+        xyz="0.096269 0 0.047551"
         rpy="0 0 0" />
       <mass
@@ -740,5 +740,5 @@
     <origin
       xyz="0 0 -0.0664"
-      rpy="-1.5708 -0.29073 1.7787E-15" />
+      rpy="-1.5708 -0.29073 0" />
     <parent
       link="${prefix}yaw_Link" />

File: dvrk_description/suj/suj.urdf.xacro (robot description, xacro)
@@ -16,5 +16,5 @@
     <inertial>
       <origin
-        xyz="3.41426483252416E-07 -0.163432953037324 0.552457766148795"
+        xyz="0 -0.163432953037324 0.552457766148795"
         rpy="0 0 0" />
       <mass
@@ -22,6 +22,6 @@
       <inertia
         ixx="116.092010218379"
-        ixy="-5.29791887754601E-06"
-        ixz="3.94601866089736E-05"
+        ixy="0"
+        ixz="0"
         iyy="116.786187825287"
         iyz="-2.79449977491914"
@@ -56,5 +56,5 @@
     <inertial>
       <origin
-        xyz="0.0568399826690053 4.20186586191917E-07 0.148466700879736"
+        xyz="0.0568399826690053 0 0.148466700879736"
         rpy="0 0 0" />
       <mass
@@ -62,8 +62,8 @@
       <inertia
         ixx="0.0849399138017183"
-        ixy="-2.62415327576062E-07"
+        ixy="0"
         ixz="-0.00950408519583723"
         iyy="0.0840388037894648"
-        iyz="-7.34496732080412E-07"
+        iyz="0"
         izz="0.0337578517914833" />
     </inertial>
@@ -114,5 +114,5 @@
     <inertial>
       <origin
-        xyz="-2.39046560324141E-06 0.181423473764042 -0.108873680906329"
+        xyz="0 0.181423473764042 -0.108873680906329"
         rpy="0 0 0" />
       <mass
@@ -120,6 +120,6 @@
       <inertia
         ixx="0.165298975805322"
-        ixy="8.05521101705082E-07"
-        ixz="1.12357011273003E-07"
+        ixy="0"
+        ixz="0"
         iyy="0.0318879130435778"
         iyz="-0.0216382058279061"
@@ -167,5 +167,5 @@
     <inertial>
       <origin
-        xyz="0.208919873467034 -5.98681643881882E-06 0.0907666144838899"
+        xyz="0.208919873467034 0 0.0907666144838899"
         rpy="0 0 0" />
       <mass
@@ -173,8 +173,8 @@
       <inertia
         ixx="0.0170495937307872"
-        ixy="1.14494065864691E-06"
+        ixy="0"
         ixz="0.0010255647636027"
         iyy="0.12264804166409"
-        iyz="-5.47956889127492E-07"
+        iyz="0"
         izz="0.114779656818464" />
     </inertial>
@@ -220,5 +220,5 @@
     <inertial>
       <origin
-        xyz="-7.80457090732156E-07 0.0671937597670209 -0.0457966340632676"
+        xyz="0 0.0671937597670209 -0.0457966340632676"
         rpy="0 0 0" />
       <mass
@@ -226,6 +226,6 @@
       <inertia
         ixx="0.00502239974642487"
-        ixy="1.37715041231818E-08"
-        ixz="6.06906568619737E-08"
+        ixy="0"
+        ixz="0"
         iyy="0.00485366592677737"
         iyz="0.000256157144769027"
@@ -273,5 +273,5 @@
     <inertial>
       <origin
-        xyz="4.481215687413E-08 0.13368960726033 0.106531287729481"
+        xyz="0 0.13368960726033 0.106531287729481"
         rpy="0 0 0" />
       <mass
@@ -279,6 +279,6 @@
       <inertia
         ixx="0.081480486654553"
-        ixy="-2.27200178709042E-08"
-        ixz="-1.15332762312484E-09"
+        ixy="0"
+        ixz="0"
         iyy="0.0179293368302569"
         iyz="-0.0218807182526152"
@@ -326,5 +326,5 @@
     <inertial>
       <origin
-        xyz="0.0568399826690054 4.20186586247429E-07 0.148466700879736"
+        xyz="0.0568399826690054 0 0.148466700879736"
         rpy="0 0 0" />
       <mass
@@ -332,8 +332,8 @@
       <inertia
         ixx="0.0849399138017188"
-        ixy="-2.62415327590614E-07"
+        ixy="0"
         ixz="-0.00950408519583733"
         iyy="0.0840388037894653"
-        iyz="-7.34496732014161E-07"
+        iyz="0"
         izz="0.0337578517914834" />
     </inertial>
@@ -367,5 +367,5 @@
     <origin
       xyz="0 0.0896 0.7611"
-      rpy="3.14159265358979 -3.41872220593534E-16 -1.5707963267949" />
+      rpy="3.14159265358979 0 -1.5707963267949" />
     <parent
       link="${prefix}base_link" />
@@ -384,5 +384,5 @@
     <inertial>
       <origin
-        xyz="-2.39046560315814E-06 -0.181423473764043 0.108873680906329"
+        xyz="0 -0.181423473764043 0.108873680906329"
         rpy="0 0 0" />
       <mass
@@ -390,6 +390,6 @@
       <inertia
         ixx="0.165298975805323"
-        ixy="-8.05521101721203E-07"
-        ixz="-1.12357011263569E-07"
+        ixy="0"
+        ixz="0"
         iyy="0.0318879130435779"
         iyz="-0.0216382058279063"
@@ -437,5 +437,5 @@
     <inertial>
       <origin
-        xyz="0.208919873467034 5.98681643856902E-06 -0.0907666144838897"
+        xyz="0.208919873467034 0 -0.0907666144838897"
         rpy="0 0 0" />
       <mass
@@ -443,8 +443,8 @@
       <inertia
         ixx="0.0170495937307872"
-        ixy="-1.14494065873328E-06"
+        ixy="0"
         ixz="-0.00102556476360276"
         iyy="0.122648041664091"
-        iyz="-5.47956889142899E-07"
+        iyz="0"
         izz="0.114779656818464" />
     </inertial>
@@ -490,5 +490,5 @@
     <inertial>
       <origin
-        xyz="0.101750929950522 0.0259124054818911 -9.32699600608711E-08"
+        xyz="0.101750929950522 0.0259124054818911 0"
         rpy="0 0 0" />
       <mass
@@ -497,7 +497,7 @@
         ixx="0.0229632930111855"
         ixy="-0.00595610077478554"
-        ixz="3.34205098594413E-08"
+        ixz="0"
         iyy="0.0229722469896469"
-        iyz="2.4231643180354E-08"
+        iyz="0"
         izz="0.0422114398260218" />
     </inertial>
@@ -543,5 +543,5 @@
     <inertial>
       <origin
-        xyz="0.056839982669005 4.20186586191917E-07 0.148466700879737"
+        xyz="0.056839982669005 0 0.148466700879737"
         rpy="0 0 0" />
       <mass
@@ -549,8 +549,8 @@
       <inertia
         ixx="0.0849399138017188"
-        ixy="-2.62415327597312E-07"
+        ixy="0"
         ixz="-0.00950408519583709"
         iyy="0.0840388037894655"
-        iyz="-7.34496732044119E-07"
+        iyz="0"
         izz="0.0337578517914837" />
     </inertial>
@@ -601,5 +601,5 @@
     <inertial>
       <origin
-        xyz="-2.39046560301936E-06 0.181423473764042 -0.108873680906329"
+        xyz="0 0.181423473764042 -0.108873680906329"
         rpy="0 0 0" />
       <mass
@@ -607,6 +607,6 @@
       <inertia
         ixx="0.165298975805321"
-        ixy="8.05521101584608E-07"
-        ixz="1.12357011233411E-07"
+        ixy="0"
+        ixz="0"
         iyy="0.0318879130435778"
         iyz="-0.0216382058279061"
@@ -654,5 +654,5 @@
     <inertial>
       <origin
-        xyz="0.208919873467034 -5.98681643837473E-06 0.0907666144838897"
+        xyz="0.208919873467034 0 0.0907666144838897"
         rpy="0 0 0" />
       <mass
@@ -660,8 +660,8 @@
       <inertia
         ixx="0.0170495937307872"
-        ixy="1.14494065865667E-06"
+        ixy="0"
         ixz="0.00102556476360271"
         iyy="0.122648041664091"
-        iyz="-5.47956889106164E-07"
+        iyz="0"
         izz="0.114779656818464" />
     </inertial>
@@ -707,5 +707,5 @@
     <inertial>
       <origin
-        xyz="-7.80457089843978E-07 -0.0671937597670209 0.0457966340632671"
+        xyz="0 -0.0671937597670209 0.0457966340632671"
         rpy="0 0 0" />
       <mass
@@ -713,6 +713,6 @@
       <inertia
         ixx="0.00502239974642493"
-        ixy="-1.37715041295868E-08"
-        ixz="-6.0690656865772E-08"
+        ixy="0"
+        ixz="0"
         iyy="0.0048536659267774"
         iyz="0.000256157144769039"
@@ -760,5 +760,5 @@
     <inertial>
       <origin
-        xyz="4.481215687413E-08 0.13368960726033 0.106531287729481"
+        xyz="0 0.13368960726033 0.106531287729481"
         rpy="0 0 0" />
       <mass
@@ -766,6 +766,6 @@
       <inertia
         ixx="0.0814804866545533"
-        ixy="-2.27200179111935E-08"
-        ixz="-1.15332763369257E-09"
+        ixy="0"
+        ixz="0"
         iyy="0.0179293368302569"
         iyz="-0.0218807182526152"
@@ -813,5 +813,5 @@
     <inertial>
       <origin
-        xyz="0.0602109648274594 -2.92606541635321E-07 0.113199880625867"
+        xyz="0.0602109648274594 0 0.113199880625867"
         rpy="0 0 0" />
       <mass
@@ -819,8 +819,8 @@
       <inertia
         ixx="0.042751844253079"
-        ixy="-6.06009647276412E-07"
+        ixy="0"
         ixz="-0.00566678005551946"
         iyy="0.0405000183180794"
-        iyz="-5.59950571967652E-07"
+        iyz="0"
         izz="0.023227300149106" />
     </inertial>
@@ -854,5 +854,5 @@
     <origin
       xyz="0 0.0895999999999999 0.3813"
-      rpy="3.14159265358979 -3.41872220593534E-16 -1.5707963267949" />
+      rpy="3.14159265358979 0 -1.5707963267949" />
     <parent
       link="${prefix}base_link" />
@@ -871,5 +871,5 @@
     <inertial>
       <origin
-        xyz="-8.83879091084783E-07 -0.269226910798469 0.0974465195036079"
+        xyz="0 -0.269226910798469 0.0974465195036079"
         rpy="0 0 0" />
       <mass
@@ -877,6 +877,6 @@
       <inertia
         ixx="0.512543337774863"
-        ixy="-1.1285325073599E-06"
-        ixz="-1.98944489031987E-07"
+        ixy="0"
+        ixz="0"
         iyy="0.046675533244729"
         iyz="-0.022324667193201"
@@ -924,5 +924,5 @@
     <inertial>
       <origin
-        xyz="0.208919873467035 -5.98681643829146E-06 0.0907666144838893"
+        xyz="0.208919873467035 0 0.0907666144838893"
         rpy="0 0 0" />
       <mass
@@ -930,8 +930,8 @@
       <inertia
         ixx="0.0170495937307872"
-        ixy="1.14494065871982E-06"
+        ixy="0"
         ixz="0.00102556476360266"
         iyy="0.122648041664091"
-        iyz="-5.47956889132769E-07"
+        iyz="0"
         izz="0.114779656818464" />
     </inertial>
@@ -977,5 +977,5 @@
     <inertial>
       <origin
-        xyz="-5.52738318171375E-07 -0.147369605966979 0.0299587011265839"
+        xyz="0 -0.147369605966979 0.0299587011265839"
         rpy="0 0 0" />
       <mass
@@ -983,6 +983,6 @@
       <inertia
         ixx="0.0128891233532759"
-        ixy="-1.05508483885794E-07"
-        ixz="2.6823702509199E-08"
+        ixy="0"
+        ixz="0"
         iyy="0.00658384974944233"
         iyz="0.00230089243299317"
@@ -1030,5 +1030,5 @@
     <inertial>
       <origin
-        xyz="4.48121568186188E-08 0.133689607260329 0.106531287729481"
+        xyz="0 0.133689607260329 0.106531287729481"
         rpy="0 0 0" />
       <mass
@@ -1036,6 +1036,6 @@
       <inertia
         ixx="0.0814804866545532"
-        ixy="-2.27200178948086E-08"
-        ixz="-1.1533276420695E-09"
+        ixy="0"
+        ixz="0"
         iyy="0.0179293368302569"
         iyz="-0.0218807182526152"

File: dvrk_description/suj/suj_launch.urdf.xacro (robot description, xacro)
@@ -1,5 +1,5 @@
 <?xml version="1.0" ?>
 <robot name="master" xmlns:xacro="http://www.ros.org/wiki/xacro">
-<xacro:include filename="$(find dvrk_description)/suj/suj.xacro"/>
+<xacro:include filename="$(find dvrk_description)/suj/suj.urdf.xacro"/>
 <xacro:suj prefix=""/>
 </robot>
