Commit message: Changed random upper case L's to lower case for links

File: dvrk_description/psm/psm.urdf.xacro (robot description, xacro)
@@ -54,5 +54,5 @@
   </link>
   <link
-    name="${prefix}yaw_Link">
+    name="${prefix}yaw_link">
     <inertial>
       <origin
@@ -75,5 +75,5 @@
       <geometry>
         <mesh
-          filename="package://dvrk_description/psm/meshes/yaw_Link.STL" />
+          filename="package://dvrk_description/psm/meshes/yaw_link.STL" />
       </geometry>
       <material
@@ -89,5 +89,5 @@
       <geometry>
         <mesh
-          filename="package://dvrk_description/psm/meshes/yaw_Link.STL" />
+          filename="package://dvrk_description/psm/meshes/yaw_link.STL" />
       </geometry>
     </collision>
@@ -102,5 +102,5 @@
       link="${prefix}base_link" />
     <child
-      link="${prefix}yaw_Link" />
+      link="${prefix}yaw_link" />
     <axis
       xyz="0 0 1" />
@@ -112,5 +112,5 @@
   </joint>
   <link
-    name="${prefix}pitch_back_Link">
+    name="${prefix}pitch_back_link">
     <inertial>
       <origin
@@ -133,5 +133,5 @@
       <geometry>
         <mesh
-          filename="package://dvrk_description/psm/meshes/pitch_back_Link.STL" />
+          filename="package://dvrk_description/psm/meshes/pitch_back_link.STL" />
       </geometry>
       <material
@@ -147,5 +147,5 @@
       <geometry>
         <mesh
-          filename="package://dvrk_description/psm/meshes/pitch_back_Link.STL" />
+          filename="package://dvrk_description/psm/meshes/pitch_back_link.STL" />
       </geometry>
     </collision>
@@ -158,7 +158,7 @@
       rpy="-1.5708 -0.29073 0" />
     <parent
-      link="${prefix}yaw_Link" />
-    <child
-      link="${prefix}pitch_back_Link" />
+      link="${prefix}yaw_link" />
+    <child
+      link="${prefix}pitch_back_link" />
     <axis
       xyz="0 0 1" />
@@ -170,5 +170,5 @@
   </joint>
   <link
-    name="${prefix}pitch_bottom_Link">
+    name="${prefix}pitch_bottom_link">
     <inertial>
       <origin
@@ -191,5 +191,5 @@
       <geometry>
         <mesh
-          filename="package://dvrk_description/psm/meshes/pitch_bottom_Link.STL" />
+          filename="package://dvrk_description/psm/meshes/pitch_bottom_link.STL" />
       </geometry>
       <material
@@ -205,5 +205,5 @@
       <geometry>
         <mesh
-          filename="package://dvrk_description/psm/meshes/pitch_bottom_Link.STL" />
+          filename="package://dvrk_description/psm/meshes/pitch_bottom_link.STL" />
       </geometry>
     </collision>
@@ -216,7 +216,7 @@
       rpy="0 0 1.8615" />
     <parent
-      link="${prefix}pitch_back_Link" />
-    <child
-      link="${prefix}pitch_bottom_Link" />
+      link="${prefix}pitch_back_link" />
+    <child
+      link="${prefix}pitch_bottom_link" />
     <axis
       xyz="0 0 1" />
@@ -229,5 +229,5 @@
   </joint>
   <link
-    name="${prefix}pitch_end_Link">
+    name="${prefix}pitch_end_link">
     <inertial>
       <origin
@@ -250,5 +250,5 @@
       <geometry>
         <mesh
-          filename="package://dvrk_description/psm/meshes/pitch_end_Link.STL" />
+          filename="package://dvrk_description/psm/meshes/pitch_end_link.STL" />
       </geometry>
       <material
@@ -264,5 +264,5 @@
       <geometry>
         <mesh
-          filename="package://dvrk_description/psm/meshes/pitch_end_Link.STL" />
+          filename="package://dvrk_description/psm/meshes/pitch_end_link.STL" />
       </geometry>
     </collision>
@@ -275,7 +275,7 @@
       rpy="0 0 0" />
     <parent
-      link="${prefix}pitch_bottom_Link" />
-    <child
-      link="${prefix}pitch_end_Link" />
+      link="${prefix}pitch_bottom_link" />
+    <child
+      link="${prefix}pitch_end_link" />
     <axis
       xyz="0 0 1" />
@@ -288,5 +288,5 @@
   </joint>
   <link
-    name="${prefix}main_insertion_Link">
+    name="${prefix}main_insertion_link">
     <inertial>
       <origin
@@ -309,5 +309,5 @@
       <geometry>
         <mesh
-          filename="package://dvrk_description/psm/meshes/main_insertion_Link.STL" />
+          filename="package://dvrk_description/psm/meshes/main_insertion_link.STL" />
       </geometry>
       <material
@@ -323,5 +323,5 @@
       <geometry>
         <mesh
-          filename="package://dvrk_description/psm/meshes/main_insertion_Link.STL" />
+          filename="package://dvrk_description/psm/meshes/main_insertion_link.STL" />
       </geometry>
     </collision>
@@ -334,7 +334,7 @@
       rpy="1.5708 1.5708 3.1416" />
     <parent
-      link="${prefix}pitch_end_Link" />
-    <child
-      link="${prefix}main_insertion_Link" />
+      link="${prefix}pitch_end_link" />
+    <child
+      link="${prefix}main_insertion_link" />
     <axis
       xyz="0 0 1" />
@@ -392,5 +392,5 @@
       rpy="0 0 -1.5708" />
     <parent
-      link="${prefix}main_insertion_Link" />
+      link="${prefix}main_insertion_link" />
     <child
       link="${prefix}tool_roll_link" />
@@ -637,5 +637,5 @@
   </joint>
   <link
-    name="${prefix}pitch_top_Link">
+    name="${prefix}pitch_top_link">
     <inertial>
       <origin
@@ -658,5 +658,5 @@
       <geometry>
         <mesh
-          filename="package://dvrk_description/psm/meshes/pitch_top_Link.STL" />
+          filename="package://dvrk_description/psm/meshes/pitch_top_link.STL" />
       </geometry>
       <material
@@ -672,5 +672,5 @@
       <geometry>
         <mesh
-          filename="package://dvrk_description/psm/meshes/pitch_top_Link.STL" />
+          filename="package://dvrk_description/psm/meshes/pitch_top_link.STL" />
       </geometry>
     </collision>
@@ -683,7 +683,7 @@
       rpy="0 0 1.8615" />
     <parent
-      link="${prefix}pitch_back_Link" />
-    <child
-      link="${prefix}pitch_top_Link" />
+      link="${prefix}pitch_back_link" />
+    <child
+      link="${prefix}pitch_top_link" />
     <axis
       xyz="0 0 1" />
@@ -696,5 +696,5 @@
   </joint>
   <link
-    name="${prefix}pitch_front_Link">
+    name="${prefix}pitch_front_link">
     <inertial>
       <origin
@@ -717,5 +717,5 @@
       <geometry>
         <mesh
-          filename="package://dvrk_description/psm/meshes/pitch_front_Link.STL" />
+          filename="package://dvrk_description/psm/meshes/pitch_front_link.STL" />
       </geometry>
       <material
@@ -731,5 +731,5 @@
       <geometry>
         <mesh
-          filename="package://dvrk_description/psm/meshes/pitch_front_Link.STL" />
+          filename="package://dvrk_description/psm/meshes/pitch_front_link.STL" />
       </geometry>
     </collision>
@@ -742,7 +742,7 @@
       rpy="-1.5708 -0.29073 0" />
     <parent
-      link="${prefix}yaw_Link" />
-    <child
-      link="${prefix}pitch_front_Link" />
+      link="${prefix}yaw_link" />
+    <child
+      link="${prefix}pitch_front_link" />
     <axis
       xyz="0 0 1" />

File: dvrk_description/psm/psm_launch.urdf.xacro (robot description, xacro)
@@ -4,4 +4,4 @@
 <link name="world"/>
 <xacro:psm parent_link="world" prefix="psm_" xyz="0 0 0.1524" rpy="0 0 0"/>
-<!--xacro:tool_lnd prefix="" parent_link="main_insertion_Link" xyz="0 0 0" rpy="0 0 0"/-->
+<!--xacro:tool_lnd prefix="" parent_link="main_insertion_link" xyz="0 0 0" rpy="0 0 0"/-->
 </robot>

Commit message: Changes in xacro and launch files

File: dvrk_description/psm/psm.urdf.xacro (robot description, xacro)
@@ -758,5 +758,5 @@
     <parent link="${prefix}base_link"/>
     <child link="${prefix}remote_center_link"/>
-    <origin rpy="0 0 0" xyz="0.4864 0 0"/>
+    <origin rpy="0 0 0" xyz="0 0.4864 0"/>
   </joint>
   </xacro:macro>
